File: keyboard_pcb/_autosave-keyboard_pcb.kicad_pcb (KiCad board)
At the start: 2 copper layers, 182 parts, among them U1 NCP1117-3.3_SOT223, U2 RP2040, U3 W25Q128JVS

Commit message: implemented LEDs and switch and diode layout
Parts:
- added LED1: MX_SK6812MINI-E, PCM_marbastlib-mx:LED_MX_6028R, B.Cu at (38.1, 33.6)
Routing:
- net Net-(D87-A): track 8.05 -> 24.3 mm
- net Net-(D84-A): track 8.05 -> 24.3 mm
- net Net-(D83-A): track 8.05 -> 24.3 mm
- net Net-(D82-A): track 8.05 -> 24.3 mm
- net Net-(D81-A): track 8.05 -> 24.3 mm
- net Net-(D80-A): track 8.05 -> 24.3 mm
- net Net-(D61-A): track 8.05 -> 24.3 mm
- net Net-(D56-A): track 8.05 -> 24.3 mm
- net Net-(D50-A): track 8.05 -> 24.3 mm
- net Net-(D43-A): track 8.05 -> 24.3 mm
- net Net-(D71-A): track 8.05 -> 24.3 mm
- net Net-(D9-A): track 8.05 -> 24.3 mm
- net Net-(D16-A): track 8.05 -> 24.3 mm
- net Net-(D12-A): track 8.05 -> 24.3 mm
- net Net-(D11-A): track 8.05 -> 24.3 mm
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Other:
- board outline added: 360 x 140 mm
