File: keyboard_pcb/LED.kicad_sch (KiCad schematic)
At the start: 87 parts

Commit message: starting routing traces part 7
Parts:
- renumbered LED30 to LED16, LED29 to LED17, LED28 to LED18, LED27 to LED19, LED26 to LED20, LED25 to LED21, LED24 to LED22, LED22 to LED24, LED21 to LED25, LED20 to LED26, LED19 to LED27, LED18 to LED28, LED17 to LED29, LED16 to LED30, LED60 to LED46, LED59 to LED47, LED58 to LED48, LED57 to LED49, LED56 to LED50, LED55 to LED51, LED54 to LED52, LED52 to LED54, LED51 to LED55, LED50 to LED56, LED49 to LED57, LED48 to LED58, LED47 to LED59, LED46 to LED60, LED87 to LED76, LED86 to LED77, LED85 to LED78, LED84 to LED79, LED83 to LED80, LED82 to LED81, LED81 to LED82, LED80 to LED83, LED79 to LED84, LED78 to LED85, LED77 to LED86, LED76 to LED87
Other:
- note added: "Hook up +5V to VDD and GND to VSS Implement debouncing capacitors"
- moved on the sheet: LED16, LED17, LED18, LED19, LED20, LED21, LED22, LED23, LED24, LED25, LED26, LED27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

Commit message: added led capacitors and route all leds
Connections:
- net +5V: now reaches LED31.1 (VDD), LED32.1 (VDD), LED33.1 (VDD), LED34.1 (VDD), LED35.1 (VDD), LED36.1 (VDD), LED37.1 (VDD), LED38.1 (VDD), LED39.1 (VDD), LED40.1 (VDD), LED41.1 (VDD), LED42.1 (VDD), LED43.1 (VDD), LED44.1 (VDD), LED45.1 (VDD)
- net +5V: now also LED1.1 (VDD), LED10.1 (VDD), LED11.1 (VDD), LED12.1 (VDD), LED13.1 (VDD), LED14.1 (VDD), LED15.1 (VDD), LED16.1 (VDD), LED17.1 (VDD), LED18.1 (VDD), LED19.1 (VDD), LED2.1 (VDD), LED20.1 (VDD), LED21.1 (VDD), LED22.1 (VDD), LED23.1 (VDD), LED24.1 (VDD), LED25.1 (VDD), LED26.1 (VDD), LED27.1 (VDD), LED28.1 (VDD), LED29.1 (VDD), LED3.1 (VDD), LED30.1 (VDD), LED4.1 (VDD), LED46.1 (VDD), LED47.1 (VDD), LED48.1 (VDD), LED49.1 (VDD), LED5.1 (VDD), LED50.1 (VDD), LED51.1 (VDD), LED52.1 (VDD), LED53.1 (VDD), LED54.1 (VDD), LED55.1 (VDD), LED56.1 (VDD), LED57.1 (VDD), LED58.1 (VDD), LED59.1 (VDD), LED6.1 (VDD), LED60.1 (VDD), LED61.1 (VDD), LED62.1 (VDD), LED63.1 (VDD), LED64.1 (VDD), LED65.1 (VDD), LED66.1 (VDD), LED67.1 (VDD), LED68.1 (VDD), LED69.1 (VDD), LED7.1 (VDD), LED70.1 (VDD), LED71.1 (VDD), LED72.1 (VDD), LED73.1 (VDD), LED74.1 (VDD), LED75.1 (VDD), LED76.1 (VDD), LED77.1 (VDD), LED78.1 (VDD), LED79.1 (VDD), LED8.1 (VDD), LED80.1 (VDD), LED81.1 (VDD), LED82.1 (VDD), LED83.1 (VDD), LED84.1 (VDD), LED85.1 (VDD), LED86.1 (VDD), LED87.1 (VDD), LED9.1 (VDD)
- net GND: now reaches LED31.4 (VSS), LED32.4 (VSS), LED33.4 (VSS), LED34.4 (VSS), LED35.4 (VSS), LED36.4 (VSS), LED37.4 (VSS), LED38.4 (VSS), LED39.4 (VSS), LED40.4 (VSS), LED41.4 (VSS), LED42.4 (VSS), LED43.4 (VSS), LED44.4 (VSS), LED45.4 (VSS)
- net GND: now also LED1.4 (VSS), LED10.4 (VSS), LED11.4 (VSS), LED12.4 (VSS), LED13.4 (VSS), LED14.4 (VSS), LED15.4 (VSS), LED16.4 (VSS), LED17.4 (VSS), LED18.4 (VSS), LED19.4 (VSS), LED2.4 (VSS), LED20.4 (VSS), LED21.4 (VSS), LED22.4 (VSS), LED23.4 (VSS), LED24.4 (VSS), LED25.4 (VSS), LED26.4 (VSS), LED27.4 (VSS), LED28.4 (VSS), LED29.4 (VSS), LED3.4 (VSS), LED30.4 (VSS), LED4.4 (VSS), LED46.4 (VSS), LED47.4 (VSS), LED48.4 (VSS), LED49.4 (VSS), LED5.4 (VSS), LED50.4 (VSS), LED51.4 (VSS), LED52.4 (VSS), LED53.4 (VSS), LED54.4 (VSS), LED55.4 (VSS), LED56.4 (VSS), LED57.4 (VSS), LED58.4 (VSS), LED59.4 (VSS), LED6.4 (VSS), LED60.4 (VSS), LED61.4 (VSS), LED62.4 (VSS), LED63.4 (VSS), LED64.4 (VSS), LED65.4 (VSS), LED66.4 (VSS), LED67.4 (VSS), LED68.4 (VSS), LED69.4 (VSS), LED7.4 (VSS), LED70.4 (VSS), LED71.4 (VSS), LED72.4 (VSS), LED73.4 (VSS), LED74.4 (VSS), LED75.4 (VSS), LED76.4 (VSS), LED77.4 (VSS), LED78.4 (VSS), LED79.4 (VSS), LED8.4 (VSS), LED80.4 (VSS), LED81.4 (VSS), LED82.4 (VSS), LED83.4 (VSS), LED84.4 (VSS), LED85.4 (VSS), LED86.4 (VSS), LED87.4 (VSS), LED9.4 (VSS)
