File: keyboard_pcb/LED.kicad_sch (KiCad schematic)
At the start: 87 parts

Commit message: relocated the mcu to the shoulder
Connections:
- net LED renamed Out_5v
Changed lines of the file:
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@@
 		)
 	)
-	(global_label "LED"
+	(global_label "Out_5v"
 		(shape input)
 		(at 40.64 40.64 180)
@@
 		)
 		(property "Intersheetrefs" "${INTERSHEET_REFS}"
-			(at 34.2077 40.64 0)
+			(at 31.3049 40.64 0)
 			(effects
 				(font
