File: keyboard_pcb/keyboard_pcb.kicad_pcb (KiCad board)
At the start: 2 copper layers, 182 parts, among them U1 NCP1117-3.3_SOT223, U2 RP2040, U3 W25Q128JVS

Commit message: update pcb with LED
Parts:
- added LED1: MX_SK6812MINI-E, PCM_marbastlib-mx:LED_MX_6028R, B.Cu at (38.1, 33.1)
- added LED10: MX_SK6812MINI-E, PCM_marbastlib-mx:LED_MX_6028R, B.Cu at (247.7, 33.1)
- added LED11: MX_SK6812MINI-E, PCM_marbastlib-mx:LED_MX_6028R, B.Cu at (266.7, 33.1)
- added LED12: MX_SK6812MINI-E, PCM_marbastlib-mx:LED_MX_6028R, B.Cu at (285.8, 33.1)
- added LED13: MX_SK6812MINI-E, PCM_marbastlib-mx:LED_MX_6028R, B.Cu at (304.8, 33.1)
- added LED14: MX_SK6812MINI-E, PCM_marbastlib-mx:LED_MX_6028R, B.Cu at (328.6, 33.1)
- added LED15: MX_SK6812MINI-E, PCM_marbastlib-mx:LED_MX_6028R, B.Cu at (347.7, 33.1)
- added LED16: MX_SK6812MINI-E, PCM_marbastlib-mx:LED_MX_6028R, B.Cu at (366.7, 33.1)
- added LED17: MX_SK6812MINI-E, PCM_marbastlib-mx:LED_MX_6028R, B.Cu at (38.1, 61.7)
- added LED18: MX_SK6812MINI-E, PCM_marbastlib-mx:LED_MX_6028R, B.Cu at (57.1, 61.7)
- added LED19: MX_SK6812MINI-E, PCM_marbastlib-mx:LED_MX_6028R, B.Cu at (76.2, 61.7)
- added LED2: MX_SK6812MINI-E, PCM_marbastlib-mx:LED_MX_6028R, B.Cu at (76.2, 33.1)
- added LED20: MX_SK6812MINI-E, PCM_marbastlib-mx:LED_MX_6028R, B.Cu at (95.2, 61.7)
- added LED21: MX_SK6812MINI-E, PCM_marbastlib-mx:LED_MX_6028R, B.Cu at (114.3, 61.7)
- added LED22: MX_SK6812MINI-E, PCM_marbastlib-mx:LED_MX_6028R, B.Cu at (133.3, 61.7)
- added LED23: MX_SK6812MINI-E, PCM_marbastlib-mx:LED_MX_6028R, B.Cu at (152.4, 61.7)
- added LED24: MX_SK6812MINI-E, PCM_marbastlib-mx:LED_MX_6028R, B.Cu at (171.4, 61.7)
- added LED25: MX_SK6812MINI-E, PCM_marbastlib-mx:LED_MX_6028R, B.Cu at (190.5, 61.7)
- added LED26: MX_SK6812MINI-E, PCM_marbastlib-mx:LED_MX_6028R, B.Cu at (209.6, 61.7)
- added LED27: MX_SK6812MINI-E, PCM_marbastlib-mx:LED_MX_6028R, B.Cu at (228.6, 61.7)
- added LED28: MX_SK6812MINI-E, PCM_marbastlib-mx:LED_MX_6028R, B.Cu at (247.7, 61.7)
- added LED29: MX_SK6812MINI-E, PCM_marbastlib-mx:LED_MX_6028R, B.Cu at (266.7, 61.7)
- added LED3: MX_SK6812MINI-E, PCM_marbastlib-mx:LED_MX_6028R, B.Cu at (95.2, 33.1)
- added LED30: MX_SK6812MINI-E, PCM_marbastlib-mx:LED_MX_6028R, B.Cu at (295.3, 61.7)
- added LED31: MX_SK6812MINI-E, PCM_marbastlib-mx:LED_MX_6028R, B.Cu at (328.6, 61.7)
- added LED32: MX_SK6812MINI-E, PCM_marbastlib-mx:LED_MX_6028R, B.Cu at (347.7, 61.7)
- added LED33: MX_SK6812MINI-E, PCM_marbastlib-mx:LED_MX_6028R, B.Cu at (366.7, 61.7)
- added LED34: MX_SK6812MINI-E, PCM_marbastlib-mx:LED_MX_6028R, B.Cu at (42.9, 80.7)
- added LED35: MX_SK6812MINI-E, PCM_marbastlib-mx:LED_MX_6028R, B.Cu at (66.7, 80.7)
- added LED36: MX_SK6812MINI-E, PCM_marbastlib-mx:LED_MX_6028R, B.Cu at (85.7, 80.7)
- added LED37: MX_SK6812MINI-E, PCM_marbastlib-mx:LED_MX_6028R, B.Cu at (104.8, 80.7)
- added LED38: MX_SK6812MINI-E, PCM_marbastlib-mx:LED_MX_6028R, B.Cu at (123.8, 80.7)
- added LED39: MX_SK6812MINI-E, PCM_marbastlib-mx:LED_MX_6028R, B.Cu at (142.9, 80.7)
- added LED4: MX_SK6812MINI-E, PCM_marbastlib-mx:LED_MX_6028R, B.Cu at (114.3, 33.1)
- added LED40: MX_SK6812MINI-E, PCM_marbastlib-mx:LED_MX_6028R, B.Cu at (161.9, 80.7)
- added LED41: MX_SK6812MINI-E, PCM_marbastlib-mx:LED_MX_6028R, B.Cu at (181.0, 80.7)
- added LED42: MX_SK6812MINI-E, PCM_marbastlib-mx:LED_MX_6028R, B.Cu at (200.0, 80.7)
- added LED43: MX_SK6812MINI-E, PCM_marbastlib-mx:LED_MX_6028R, B.Cu at (219.1, 80.7)
- added LED44: MX_SK6812MINI-E, PCM_marbastlib-mx:LED_MX_6028R, B.Cu at (238.1, 80.7)
- added LED45: MX_SK6812MINI-E, PCM_marbastlib-mx:LED_MX_6028R, B.Cu at (257.2, 80.7)
- added LED46: MX_SK6812MINI-E, PCM_marbastlib-mx:LED_MX_6028R, B.Cu at (276.2, 80.7)
- added LED47: MX_SK6812MINI-E, PCM_marbastlib-mx:LED_MX_6028R, B.Cu at (300.0, 80.7)
- added LED48: MX_SK6812MINI-E, PCM_marbastlib-mx:LED_MX_6028R, B.Cu at (328.6, 80.7)
- added LED49: MX_SK6812MINI-E, PCM_marbastlib-mx:LED_MX_6028R, B.Cu at (347.7, 80.7)
- added LED5: MX_SK6812MINI-E, PCM_marbastlib-mx:LED_MX_6028R, B.Cu at (133.3, 33.1)
- added LED50: MX_SK6812MINI-E, PCM_marbastlib-mx:LED_MX_6028R, B.Cu at (366.7, 80.7)
- added LED51: MX_SK6812MINI-E, PCM_marbastlib-mx:LED_MX_6028R, B.Cu at (45.2, 99.8)
- added LED52: MX_SK6812MINI-E, PCM_marbastlib-mx:LED_MX_6028R, B.Cu at (71.4, 99.8)
- added LED53: MX_SK6812MINI-E, PCM_marbastlib-mx:LED_MX_6028R, B.Cu at (90.5, 99.8)
- added LED54: MX_SK6812MINI-E, PCM_marbastlib-mx:LED_MX_6028R, B.Cu at (109.5, 99.8)
- added LED55: MX_SK6812MINI-E, PCM_marbastlib-mx:LED_MX_6028R, B.Cu at (128.6, 99.8)
- added LED56: MX_SK6812MINI-E, PCM_marbastlib-mx:LED_MX_6028R, B.Cu at (147.6, 99.8)
- added LED57: MX_SK6812MINI-E, PCM_marbastlib-mx:LED_MX_6028R, B.Cu at (166.7, 99.8)
- added LED58: MX_SK6812MINI-E, PCM_marbastlib-mx:LED_MX_6028R, B.Cu at (185.7, 99.8)
- added LED59: MX_SK6812MINI-E, PCM_marbastlib-mx:LED_MX_6028R, B.Cu at (204.8, 99.8)
- added LED6: MX_SK6812MINI-E, PCM_marbastlib-mx:LED_MX_6028R, B.Cu at (161.9, 33.1)
- added LED60: MX_SK6812MINI-E, PCM_marbastlib-mx:LED_MX_6028R, B.Cu at (223.8, 99.8)
- added LED61: MX_SK6812MINI-E, PCM_marbastlib-mx:LED_MX_6028R, B.Cu at (242.9, 99.8)
- added LED62: MX_SK6812MINI-E, PCM_marbastlib-mx:LED_MX_6028R, B.Cu at (261.9, 99.8)
- added LED63: MX_SK6812MINI-E, PCM_marbastlib-mx:LED_MX_6028R, B.Cu at (292.9, 99.8)
- added LED64: MX_SK6812MINI-E, PCM_marbastlib-mx:LED_MX_6028R, B.Cu at (50.0, 118.8)
- added LED65: MX_SK6812MINI-E, PCM_marbastlib-mx:LED_MX_6028R, B.Cu at (81.0, 118.8)
- added LED66: MX_SK6812MINI-E, PCM_marbastlib-mx:LED_MX_6028R, B.Cu at (100.0, 118.8)
- added LED67: MX_SK6812MINI-E, PCM_marbastlib-mx:LED_MX_6028R, B.Cu at (119.1, 118.8)
- added LED68: MX_SK6812MINI-E, PCM_marbastlib-mx:LED_MX_6028R, B.Cu at (138.1, 118.8)
- added LED69: MX_SK6812MINI-E, PCM_marbastlib-mx:LED_MX_6028R, B.Cu at (157.2, 118.8)
- added LED7: MX_SK6812MINI-E, PCM_marbastlib-mx:LED_MX_6028R, B.Cu at (181.0, 33.1)
- added LED70: MX_SK6812MINI-E, PCM_marbastlib-mx:LED_MX_6028R, B.Cu at (176.2, 118.8)
- added LED71: MX_SK6812MINI-E, PCM_marbastlib-mx:LED_MX_6028R, B.Cu at (195.3, 118.8)
- added LED72: MX_SK6812MINI-E, PCM_marbastlib-mx:LED_MX_6028R, B.Cu at (214.3, 118.8)
- added LED73: MX_SK6812MINI-E, PCM_marbastlib-mx:LED_MX_6028R, B.Cu at (233.4, 118.8)
- added LED74: MX_SK6812MINI-E, PCM_marbastlib-mx:LED_MX_6028R, B.Cu at (252.4, 118.8)
- added LED75: MX_SK6812MINI-E, PCM_marbastlib-mx:LED_MX_6028R, B.Cu at (288.1, 118.8)
- added LED76: MX_SK6812MINI-E, PCM_marbastlib-mx:LED_MX_6028R, B.Cu at (347.7, 118.8)
- added LED77: MX_SK6812MINI-E, PCM_marbastlib-mx:LED_MX_6028R, B.Cu at (40.5, 137.9)
- added LED78: MX_SK6812MINI-E, PCM_marbastlib-mx:LED_MX_6028R, B.Cu at (64.3, 137.9)
- added LED79: MX_SK6812MINI-E, PCM_marbastlib-mx:LED_MX_6028R, B.Cu at (88.1, 137.9)
- added LED8: MX_SK6812MINI-E, PCM_marbastlib-mx:LED_MX_6028R, B.Cu at (200.0, 33.1)
- added LED80: MX_SK6812MINI-E, PCM_marbastlib-mx:LED_MX_6028R, B.Cu at (159.5, 137.9)
- added LED81: MX_SK6812MINI-E, PCM_marbastlib-mx:LED_MX_6028R, B.Cu at (231.0, 137.9)
- added LED82: MX_SK6812MINI-E, PCM_marbastlib-mx:LED_MX_6028R, B.Cu at (254.8, 137.9)
- added LED83: MX_SK6812MINI-E, PCM_marbastlib-mx:LED_MX_6028R, B.Cu at (278.6, 137.9)
- added LED84: MX_SK6812MINI-E, PCM_marbastlib-mx:LED_MX_6028R, B.Cu at (302.4, 137.9)
- added LED85: MX_SK6812MINI-E, PCM_marbastlib-mx:LED_MX_6028R, B.Cu at (328.6, 137.9)
- added LED86: MX_SK6812MINI-E, PCM_marbastlib-mx:LED_MX_6028R, B.Cu at (347.7, 137.9)
- added LED87: MX_SK6812MINI-E, PCM_marbastlib-mx:LED_MX_6028R, B.Cu at (366.7, 137.9)
- added LED9: MX_SK6812MINI-E, PCM_marbastlib-mx:LED_MX_6028R, B.Cu at (219.1, 33.1)
Routing:
- net Net-(D87-A): track 8.05 -> 52.9 mm
- net Net-(D84-A): track 8.05 -> 52.9 mm
- net Net-(D83-A): track 8.05 -> 52.9 mm
- net Net-(D82-A): track 8.05 -> 52.9 mm
- net Net-(D81-A): track 8.05 -> 52.9 mm
- net Net-(D80-A): track 8.05 -> 52.9 mm
- net Net-(D61-A): track 8.05 -> 52.9 mm
- net Net-(D56-A): track 8.05 -> 52.9 mm
- net Net-(D50-A): track 8.05 -> 52.9 mm
- net Net-(D43-A): track 8.05 -> 52.9 mm
- net Net-(D71-A): track 8.05 -> 52.9 mm
- net Net-(D9-A): track 8.05 -> 52.9 mm
- net Net-(D16-A): track 8.05 -> 52.9 mm
- net Net-(D12-A): track 8.05 -> 52.9 mm
- net Net-(D11-A): track 8.05 -> 52.9 mm
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Other:
- board outline added: 360 x 140 mm

Commit message: starting routing traces part 7
Parts:
- moved LED77 307.2 mm to (40.5, 137.9)
- moved LED86 307.2 mm to (347.7, 137.9)
- moved LED78 264.3 mm to (64.3, 137.9)
- moved LED85 264.3 mm to (328.6, 137.9)
- moved LED17 228.6 mm to (38.1, 61.7)
- moved LED29 228.6 mm to (266.7, 61.7)
- moved LED50 219.9 mm to (366.7, 80.7)
- moved LED56 219.9 mm to (147.6, 99.8)
- moved LED79 214.3 mm to (88.1, 137.9)
- moved LED84 214.3 mm to (302.4, 137.9)
- moved LED18 190.5 mm to (57.1, 61.7)
- moved LED28 190.5 mm to (247.7, 61.7)
- moved LED49 182.0 mm to (347.7, 80.7)
- moved LED57 182.0 mm to (166.7, 99.8)
- moved LED19 152.4 mm to (76.2, 61.7)
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- renumbered LED30 to LED16, LED29 to LED17, LED28 to LED18, LED27 to LED19, LED26 to LED20, LED25 to LED21, LED24 to LED22, LED22 to LED24, LED21 to LED25, LED20 to LED26, LED19 to LED27, LED18 to LED28, LED17 to LED29, LED16 to LED30, LED60 to LED46, LED59 to LED47, LED58 to LED48, LED57 to LED49, LED56 to LED50, LED55 to LED51, LED54 to LED52, LED52 to LED54, LED51 to LED55, LED50 to LED56, LED49 to LED57, LED48 to LED58, LED47 to LED59, LED46 to LED60, LED87 to LED76, LED86 to LED77, LED85 to LED78, LED84 to LED79, LED83 to LED80, LED82 to LED81, LED81 to LED82, LED80 to LED83, LED79 to LED84, LED78 to LED85, LED77 to LED86, LED76 to LED87
Connections:
- MX52 pad 1: col2 -> col1
Routing:
- net Net-(LED76-VSS): track 0.00 -> 356.6 mm
- net row1: track 0.00 -> 341.1 mm
- net row0: track 0.00 -> 340.4 mm
- net row2: track 0.00 -> 336.4 mm
- net row5: track 0.00 -> 334.2 mm
- net Net-(LED1-VDD): track 0.00 -> 328.9 mm
- net Net-(LED76-VDD): track 0.00 -> 327.8 mm
- net row4: track 0.00 -> 307.0 mm
- net row3: track 0.00 -> 257.1 mm
- net col7: track 0.00 -> 129.8 mm
- net col12: track 0.00 -> 129.4 mm
- net col10: track 0.00 -> 128.1 mm
- net col11: track 0.00 -> 127.5 mm
- net col13: track 0.00 -> 127.2 mm
- net col2: track 0.00 -> 115.6 mm
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
Commit message: added led capacitors and route all leds
Parts:
- added C1: 100nF, Capacitor_SMD:C_0603_1608Metric_Pad1.08x0.95mm_HandSolder, B.Cu at (44.1, 33.9)
- added C10: 100nF, Capacitor_SMD:C_0603_1608Metric_Pad1.08x0.95mm_HandSolder, B.Cu at (253.7, 33.9)
- added C100: 100nF, Capacitor_SMD:C_0603_1608Metric_Pad1.08x0.95mm_HandSolder, F.Cu at (-92.9, 61.0)
- added C101: 10u, Capacitor_SMD:C_0603_1608Metric_Pad1.08x0.95mm_HandSolder, F.Cu at (-92.9, 64.3)
- added C102: 30pF, Capacitor_SMD:C_0603_1608Metric_Pad1.08x0.95mm_HandSolder, F.Cu at (-92.9, 67.7)
- added C103: 30pF, Capacitor_SMD:C_0603_1608Metric_Pad1.08x0.95mm_HandSolder, F.Cu at (-92.9, 71.0)
- added C104: 100nF, Capacitor_SMD:C_0603_1608Metric_Pad1.08x0.95mm_HandSolder, F.Cu at (-92.9, 74.4)
- added C11: 100nF, Capacitor_SMD:C_0603_1608Metric_Pad1.08x0.95mm_HandSolder, B.Cu at (272.7, 33.9)
- added C12: 100nF, Capacitor_SMD:C_0603_1608Metric_Pad1.08x0.95mm_HandSolder, B.Cu at (291.8, 33.9)
- added C13: 100nF, Capacitor_SMD:C_0603_1608Metric_Pad1.08x0.95mm_HandSolder, B.Cu at (310.8, 33.9)
- added C14: 100nF, Capacitor_SMD:C_0603_1608Metric_Pad1.08x0.95mm_HandSolder, B.Cu at (334.6, 33.9)
- added C15: 100nF, Capacitor_SMD:C_0603_1608Metric_Pad1.08x0.95mm_HandSolder, B.Cu at (353.7, 33.9)
- added C16: 100nF, Capacitor_SMD:C_0603_1608Metric_Pad1.08x0.95mm_HandSolder, B.Cu at (372.7, 33.9)
- added C17: 100nF, Capacitor_SMD:C_0603_1608Metric_Pad1.08x0.95mm_HandSolder, B.Cu at (44.1, 62.4)
- added C18: 100nF, Capacitor_SMD:C_0603_1608Metric_Pad1.08x0.95mm_HandSolder, B.Cu at (63.1, 62.4)
- added C19: 100nF, Capacitor_SMD:C_0603_1608Metric_Pad1.08x0.95mm_HandSolder, B.Cu at (82.2, 62.4)
- added C2: 100nF, Capacitor_SMD:C_0603_1608Metric_Pad1.08x0.95mm_HandSolder, B.Cu at (82.2, 33.9)
- added C20: 100nF, Capacitor_SMD:C_0603_1608Metric_Pad1.08x0.95mm_HandSolder, B.Cu at (101.2, 62.4)
- added C21: 100nF, Capacitor_SMD:C_0603_1608Metric_Pad1.08x0.95mm_HandSolder, B.Cu at (120.3, 62.4)
- added C22: 100nF, Capacitor_SMD:C_0603_1608Metric_Pad1.08x0.95mm_HandSolder, B.Cu at (139.3, 62.4)
- added C23: 100nF, Capacitor_SMD:C_0603_1608Metric_Pad1.08x0.95mm_HandSolder, B.Cu at (158.4, 62.4)
- added C24: 100nF, Capacitor_SMD:C_0603_1608Metric_Pad1.08x0.95mm_HandSolder, B.Cu at (177.4, 62.4)
- added C25: 100nF, Capacitor_SMD:C_0603_1608Metric_Pad1.08x0.95mm_HandSolder, B.Cu at (196.5, 62.4)
- added C26: 100nF, Capacitor_SMD:C_0603_1608Metric_Pad1.08x0.95mm_HandSolder, B.Cu at (215.6, 62.4)
- added C27: 100nF, Capacitor_SMD:C_0603_1608Metric_Pad1.08x0.95mm_HandSolder, B.Cu at (234.6, 62.4)
- added C28: 100nF, Capacitor_SMD:C_0603_1608Metric_Pad1.08x0.95mm_HandSolder, B.Cu at (253.7, 62.4)
- added C29: 100nF, Capacitor_SMD:C_0603_1608Metric_Pad1.08x0.95mm_HandSolder, B.Cu at (272.7, 62.4)
- added C3: 100nF, Capacitor_SMD:C_0603_1608Metric_Pad1.08x0.95mm_HandSolder, B.Cu at (101.2, 33.9)
- added C30: 100nF, Capacitor_SMD:C_0603_1608Metric_Pad1.08x0.95mm_HandSolder, B.Cu at (301.3, 62.4)
- added C31: 100nF, Capacitor_SMD:C_0603_1608Metric_Pad1.08x0.95mm_HandSolder, B.Cu at (334.6, 62.4)
- added C32: 100nF, Capacitor_SMD:C_0603_1608Metric_Pad1.08x0.95mm_HandSolder, B.Cu at (353.7, 62.4)
- added C33: 100nF, Capacitor_SMD:C_0603_1608Metric_Pad1.08x0.95mm_HandSolder, B.Cu at (372.7, 62.4)
- added C34: 100nF, Capacitor_SMD:C_0603_1608Metric_Pad1.08x0.95mm_HandSolder, B.Cu at (48.9, 81.5)
- added C35: 100nF, Capacitor_SMD:C_0603_1608Metric_Pad1.08x0.95mm_HandSolder, B.Cu at (72.7, 81.5)
- added C36: 100nF, Capacitor_SMD:C_0603_1608Metric_Pad1.08x0.95mm_HandSolder, B.Cu at (91.7, 81.5)
- added C37: 100nF, Capacitor_SMD:C_0603_1608Metric_Pad1.08x0.95mm_HandSolder, B.Cu at (110.8, 81.5)
- added C38: 100nF, Capacitor_SMD:C_0603_1608Metric_Pad1.08x0.95mm_HandSolder, B.Cu at (129.8, 81.5)
- added C39: 100nF, Capacitor_SMD:C_0603_1608Metric_Pad1.08x0.95mm_HandSolder, B.Cu at (148.9, 81.5)
- added C4: 100nF, Capacitor_SMD:C_0603_1608Metric_Pad1.08x0.95mm_HandSolder, B.Cu at (120.3, 33.9)
- added C40: 100nF, Capacitor_SMD:C_0603_1608Metric_Pad1.08x0.95mm_HandSolder, B.Cu at (167.9, 81.5)
- added C41: 100nF, Capacitor_SMD:C_0603_1608Metric_Pad1.08x0.95mm_HandSolder, B.Cu at (187.0, 81.5)
- added C42: 100nF, Capacitor_SMD:C_0603_1608Metric_Pad1.08x0.95mm_HandSolder, B.Cu at (206.0, 81.5)
- added C43: 100nF, Capacitor_SMD:C_0603_1608Metric_Pad1.08x0.95mm_HandSolder, B.Cu at (225.1, 81.5)
- added C44: 100nF, Capacitor_SMD:C_0603_1608Metric_Pad1.08x0.95mm_HandSolder, B.Cu at (244.1, 81.5)
- added C45: 100nF, Capacitor_SMD:C_0603_1608Metric_Pad1.08x0.95mm_HandSolder, B.Cu at (263.2, 81.5)
- added C46: 100nF, Capacitor_SMD:C_0603_1608Metric_Pad1.08x0.95mm_HandSolder, B.Cu at (282.2, 81.5)
- added C47: 100nF, Capacitor_SMD:C_0603_1608Metric_Pad1.08x0.95mm_HandSolder, B.Cu at (306.0, 81.5)
- added C48: 100nF, Capacitor_SMD:C_0603_1608Metric_Pad1.08x0.95mm_HandSolder, B.Cu at (334.6, 81.5)
- added C49: 100nF, Capacitor_SMD:C_0603_1608Metric_Pad1.08x0.95mm_HandSolder, B.Cu at (353.7, 81.5)
- added C5: 100nF, Capacitor_SMD:C_0603_1608Metric_Pad1.08x0.95mm_HandSolder, B.Cu at (139.3, 33.9)
- added C50: 100nF, Capacitor_SMD:C_0603_1608Metric_Pad1.08x0.95mm_HandSolder, B.Cu at (372.7, 81.5)
- added C51: 100nF, Capacitor_SMD:C_0603_1608Metric_Pad1.08x0.95mm_HandSolder, B.Cu at (51.2, 100.5)
- added C52: 100nF, Capacitor_SMD:C_0603_1608Metric_Pad1.08x0.95mm_HandSolder, B.Cu at (77.4, 100.5)
- added C53: 100nF, Capacitor_SMD:C_0603_1608Metric_Pad1.08x0.95mm_HandSolder, B.Cu at (96.5, 100.5)
- added C54: 100nF, Capacitor_SMD:C_0603_1608Metric_Pad1.08x0.95mm_HandSolder, B.Cu at (115.5, 100.5)
- added C55: 100nF, Capacitor_SMD:C_0603_1608Metric_Pad1.08x0.95mm_HandSolder, B.Cu at (134.6, 100.5)
- added C56: 100nF, Capacitor_SMD:C_0603_1608Metric_Pad1.08x0.95mm_HandSolder, B.Cu at (153.6, 100.5)
- added C57: 100nF, Capacitor_SMD:C_0603_1608Metric_Pad1.08x0.95mm_HandSolder, B.Cu at (172.7, 100.5)
- added C58: 100nF, Capacitor_SMD:C_0603_1608Metric_Pad1.08x0.95mm_HandSolder, B.Cu at (191.7, 100.5)
- added C59: 100nF, Capacitor_SMD:C_0603_1608Metric_Pad1.08x0.95mm_HandSolder, B.Cu at (210.8, 100.5)
- added C6: 100nF, Capacitor_SMD:C_0603_1608Metric_Pad1.08x0.95mm_HandSolder, B.Cu at (167.9, 33.9)
- added C60: 100nF, Capacitor_SMD:C_0603_1608Metric_Pad1.08x0.95mm_HandSolder, B.Cu at (229.8, 100.5)
- added C61: 100nF, Capacitor_SMD:C_0603_1608Metric_Pad1.08x0.95mm_HandSolder, B.Cu at (248.9, 100.5)
- added C62: 100nF, Capacitor_SMD:C_0603_1608Metric_Pad1.08x0.95mm_HandSolder, B.Cu at (267.9, 100.5)
- added C63: 100nF, Capacitor_SMD:C_0603_1608Metric_Pad1.08x0.95mm_HandSolder, B.Cu at (298.9, 100.5)
- added C64: 100nF, Capacitor_SMD:C_0603_1608Metric_Pad1.08x0.95mm_HandSolder, B.Cu at (56.0, 119.6)
- added C65: 100nF, Capacitor_SMD:C_0603_1608Metric_Pad1.08x0.95mm_HandSolder, B.Cu at (87.0, 119.6)
- added C66: 100nF, Capacitor_SMD:C_0603_1608Metric_Pad1.08x0.95mm_HandSolder, B.Cu at (106.0, 119.6)
- added C67: 100nF, Capacitor_SMD:C_0603_1608Metric_Pad1.08x0.95mm_HandSolder, B.Cu at (125.1, 119.6)
- added C68: 100nF, Capacitor_SMD:C_0603_1608Metric_Pad1.08x0.95mm_HandSolder, B.Cu at (144.1, 119.6)
- added C69: 100nF, Capacitor_SMD:C_0603_1608Metric_Pad1.08x0.95mm_HandSolder, B.Cu at (163.2, 119.6)
- added C7: 100nF, Capacitor_SMD:C_0603_1608Metric_Pad1.08x0.95mm_HandSolder, B.Cu at (187.0, 33.9)
- added C70: 100nF, Capacitor_SMD:C_0603_1608Metric_Pad1.08x0.95mm_HandSolder, B.Cu at (182.2, 119.6)
- added C71: 100nF, Capacitor_SMD:C_0603_1608Metric_Pad1.08x0.95mm_HandSolder, B.Cu at (201.3, 119.6)
- added C72: 100nF, Capacitor_SMD:C_0603_1608Metric_Pad1.08x0.95mm_HandSolder, B.Cu at (220.3, 119.6)
- added C73: 100nF, Capacitor_SMD:C_0603_1608Metric_Pad1.08x0.95mm_HandSolder, B.Cu at (239.4, 119.6)
- added C74: 100nF, Capacitor_SMD:C_0603_1608Metric_Pad1.08x0.95mm_HandSolder, B.Cu at (258.4, 119.6)
- added C75: 100nF, Capacitor_SMD:C_0603_1608Metric_Pad1.08x0.95mm_HandSolder, B.Cu at (294.1, 119.6)
- added C76: 100nF, Capacitor_SMD:C_0603_1608Metric_Pad1.08x0.95mm_HandSolder, B.Cu at (353.7, 119.6)
- added C77: 100nF, Capacitor_SMD:C_0603_1608Metric_Pad1.08x0.95mm_HandSolder, B.Cu at (46.5, 138.6)
- added C78: 100nF, Capacitor_SMD:C_0603_1608Metric_Pad1.08x0.95mm_HandSolder, B.Cu at (70.3, 138.6)
- added C79: 100nF, Capacitor_SMD:C_0603_1608Metric_Pad1.08x0.95mm_HandSolder, B.Cu at (94.1, 138.6)
- added C8: 100nF, Capacitor_SMD:C_0603_1608Metric_Pad1.08x0.95mm_HandSolder, B.Cu at (206.0, 33.9)
- added C80: 100nF, Capacitor_SMD:C_0603_1608Metric_Pad1.08x0.95mm_HandSolder, B.Cu at (165.5, 138.6)
- added C81: 100nF, Capacitor_SMD:C_0603_1608Metric_Pad1.08x0.95mm_HandSolder, B.Cu at (237.0, 138.6)
- added C82: 100nF, Capacitor_SMD:C_0603_1608Metric_Pad1.08x0.95mm_HandSolder, B.Cu at (260.8, 138.6)
- added C83: 100nF, Capacitor_SMD:C_0603_1608Metric_Pad1.08x0.95mm_HandSolder, B.Cu at (284.6, 138.6)
- added C84: 100nF, Capacitor_SMD:C_0603_1608Metric_Pad1.08x0.95mm_HandSolder, B.Cu at (308.4, 138.6)
- added C85: 100nF, Capacitor_SMD:C_0603_1608Metric_Pad1.08x0.95mm_HandSolder, B.Cu at (334.6, 138.6)
- added C86: 100nF, Capacitor_SMD:C_0603_1608Metric_Pad1.08x0.95mm_HandSolder, B.Cu at (353.7, 138.6)
- added C87: 100nF, Capacitor_SMD:C_0603_1608Metric_Pad1.08x0.95mm_HandSolder, B.Cu at (372.7, 138.6)
- added C88: 100nF, Capacitor_SMD:C_0603_1608Metric_Pad1.08x0.95mm_HandSolder, F.Cu at (-104.9, 61.0)
- added C89: 100nF, Capacitor_SMD:C_0603_1608Metric_Pad1.08x0.95mm_HandSolder, F.Cu at (-104.9, 64.3)
- added C9: 100nF, Capacitor_SMD:C_0603_1608Metric_Pad1.08x0.95mm_HandSolder, B.Cu at (225.1, 33.9)
- added C90: 100nF, Capacitor_SMD:C_0603_1608Metric_Pad1.08x0.95mm_HandSolder, F.Cu at (-104.9, 67.7)
- added C91: 100nF, Capacitor_SMD:C_0603_1608Metric_Pad1.08x0.95mm_HandSolder, F.Cu at (-104.9, 71.0)
- added C92: 100nF, Capacitor_SMD:C_0603_1608Metric_Pad1.08x0.95mm_HandSolder, F.Cu at (-104.9, 74.4)
- added C93: 100nF, Capacitor_SMD:C_0603_1608Metric_Pad1.08x0.95mm_HandSolder, F.Cu at (-104.9, 77.7)
- added C94: 100nF, Capacitor_SMD:C_0603_1608Metric_Pad1.08x0.95mm_HandSolder, F.Cu at (-98.9, 61.0)
- added C95: 100nF, Capacitor_SMD:C_0603_1608Metric_Pad1.08x0.95mm_HandSolder, F.Cu at (-98.9, 64.3)
- added C96: 100nF, Capacitor_SMD:C_0603_1608Metric_Pad1.08x0.95mm_HandSolder, F.Cu at (-98.9, 67.7)
- added C97: 1uF, Capacitor_SMD:C_0603_1608Metric_Pad1.08x0.95mm_HandSolder, F.Cu at (-98.9, 71.0)
- added C98: 1uF, Capacitor_SMD:C_0603_1608Metric_Pad1.08x0.95mm_HandSolder, F.Cu at (-98.9, 74.4)
- added C99: 10u, Capacitor_SMD:C_0603_1608Metric_Pad1.08x0.95mm_HandSolder, F.Cu at (-98.9, 77.7)
- renumbered S6 to S1, S3 to S2, S2 to S3, S5 to S4, S1 to S5
Connections:
- LED1 pad 1: Net-(LED1-VDD) -> +5V
- LED1 pad 4: Net-(LED1-VSS) -> GND
- LED10 pad 1: Net-(LED1-VDD) -> +5V
- LED10 pad 4: Net-(LED1-VSS) -> GND
- LED11 pad 1: Net-(LED1-VDD) -> +5V
- LED11 pad 4: Net-(LED1-VSS) -> GND
- LED12 pad 1: Net-(LED1-VDD) -> +5V
- LED12 pad 4: Net-(LED1-VSS) -> GND
- LED13 pad 1: Net-(LED1-VDD) -> +5V
- LED13 pad 4: Net-(LED1-VSS) -> GND
- LED14 pad 1: Net-(LED1-VDD) -> +5V
- LED14 pad 4: Net-(LED1-VSS) -> GND
- LED15 pad 1: Net-(LED1-VDD) -> +5V
- LED15 pad 4: Net-(LED1-VSS) -> GND
- LED16 pad 1: Net-(LED16-VDD) -> +5V
- LED16 pad 4: Net-(LED16-VSS) -> GND
- LED17 pad 1: Net-(LED16-VDD) -> +5V
- LED17 pad 4: Net-(LED16-VSS) -> GND
- LED18 pad 1: Net-(LED16-VDD) -> +5V
- LED18 pad 4: Net-(LED16-VSS) -> GND
- LED19 pad 1: Net-(LED16-VDD) -> +5V
- LED19 pad 4: Net-(LED16-VSS) -> GND
- LED2 pad 1: Net-(LED1-VDD) -> +5V
- LED2 pad 4: Net-(LED1-VSS) -> GND
- LED20 pad 1: Net-(LED16-VDD) -> +5V
- LED20 pad 4: Net-(LED16-VSS) -> GND
- LED21 pad 1: Net-(LED16-VDD) -> +5V
- LED21 pad 4: Net-(LED16-VSS) -> GND
- LED22 pad 1: Net-(LED16-VDD) -> +5V
- LED22 pad 4: Net-(LED16-VSS) -> GND
- LED23 pad 1: Net-(LED16-VDD) -> +5V
- LED23 pad 4: Net-(LED16-VSS) -> GND
- LED24 pad 1: Net-(LED16-VDD) -> +5V
- LED24 pad 4: Net-(LED16-VSS) -> GND
- LED25 pad 1: Net-(LED16-VDD) -> +5V
- LED25 pad 4: Net-(LED16-VSS) -> GND
- LED26 pad 1: Net-(LED16-VDD) -> +5V
- LED26 pad 4: Net-(LED16-VSS) -> GND
- LED27 pad 1: Net-(LED16-VDD) -> +5V
- LED27 pad 4: Net-(LED16-VSS) -> GND
- LED28 pad 1: Net-(LED16-VDD) -> +5V
- LED28 pad 4: Net-(LED16-VSS) -> GND
- LED29 pad 1: Net-(LED16-VDD) -> +5V
- LED29 pad 4: Net-(LED16-VSS) -> GND
- LED3 pad 1: Net-(LED1-VDD) -> +5V
- LED3 pad 4: Net-(LED1-VSS) -> GND
- LED30 pad 1: Net-(LED16-VDD) -> +5V
- LED30 pad 4: Net-(LED16-VSS) -> GND
- LED31 pad 1: Net-(LED31-VDD) -> +5V
- LED31 pad 4: Net-(LED31-VSS) -> GND
- LED32 pad 1: Net-(LED31-VDD) -> +5V
- LED32 pad 4: Net-(LED31-VSS) -> GND
- LED33 pad 1: Net-(LED31-VDD) -> +5V
- LED33 pad 4: Net-(LED31-VSS) -> GND
- LED34 pad 1: Net-(LED31-VDD) -> +5V
- LED34 pad 4: Net-(LED31-VSS) -> GND
- LED35 pad 1: Net-(LED31-VDD) -> +5V
- LED35 pad 4: Net-(LED31-VSS) -> GND
- LED36 pad 1: Net-(LED31-VDD) -> +5V
- LED36 pad 4: Net-(LED31-VSS) -> GND
- LED37 pad 1: Net-(LED31-VDD) -> +5V
- LED37 pad 4: Net-(LED31-VSS) -> GND
- LED38 pad 1: Net-(LED31-VDD) -> +5V
- LED38 pad 4: Net-(LED31-VSS) -> GND
- LED39 pad 1: Net-(LED31-VDD) -> +5V
- LED39 pad 4: Net-(LED31-VSS) -> GND
- LED4 pad 1: Net-(LED1-VDD) -> +5V
- LED4 pad 4: Net-(LED1-VSS) -> GND
- LED40 pad 1: Net-(LED31-VDD) -> +5V
- LED40 pad 4: Net-(LED31-VSS) -> GND
- LED41 pad 1: Net-(LED31-VDD) -> +5V
- LED41 pad 4: Net-(LED31-VSS) -> GND
- LED42 pad 1: Net-(LED31-VDD) -> +5V
- LED42 pad 4: Net-(LED31-VSS) -> GND
- LED43 pad 1: Net-(LED31-VDD) -> +5V
- LED43 pad 4: Net-(LED31-VSS) -> GND
- LED44 pad 1: Net-(LED31-VDD) -> +5V
- LED44 pad 4: Net-(LED31-VSS) -> GND
- LED45 pad 1: Net-(LED31-VDD) -> +5V
- LED45 pad 4: Net-(LED31-VSS) -> GND
- LED46 pad 1: Net-(LED46-VDD) -> +5V
- LED46 pad 4: Net-(LED46-VSS) -> GND
- LED47 pad 1: Net-(LED46-VDD) -> +5V
- LED47 pad 4: Net-(LED46-VSS) -> GND
- LED48 pad 1: Net-(LED46-VDD) -> +5V
- LED48 pad 4: Net-(LED46-VSS) -> GND
- LED49 pad 1: Net-(LED46-VDD) -> +5V
- LED49 pad 4: Net-(LED46-VSS) -> GND
- LED5 pad 1: Net-(LED1-VDD) -> +5V
- LED5 pad 4: Net-(LED1-VSS) -> GND
- LED50 pad 1: Net-(LED46-VDD) -> +5V
- LED50 pad 4: Net-(LED46-VSS) -> GND
- LED51 pad 1: Net-(LED46-VDD) -> +5V
- LED51 pad 4: Net-(LED46-VSS) -> GND
- LED52 pad 1: Net-(LED46-VDD) -> +5V
- LED52 pad 4: Net-(LED46-VSS) -> GND
- LED53 pad 1: Net-(LED46-VDD) -> +5V
- LED53 pad 4: Net-(LED46-VSS) -> GND
- LED54 pad 1: Net-(LED46-VDD) -> +5V
- LED54 pad 4: Net-(LED46-VSS) -> GND
- LED55 pad 1: Net-(LED46-VDD) -> +5V
- LED55 pad 4: Net-(LED46-VSS) -> GND
- LED56 pad 1: Net-(LED46-VDD) -> +5V
- LED56 pad 4: Net-(LED46-VSS) -> GND
- LED57 pad 1: Net-(LED46-VDD) -> +5V
- LED57 pad 4: Net-(LED46-VSS) -> GND
- LED58 pad 1: Net-(LED46-VDD) -> +5V
- LED58 pad 4: Net-(LED46-VSS) -> GND
- LED59 pad 1: Net-(LED46-VDD) -> +5V
- LED59 pad 4: Net-(LED46-VSS) -> GND
- LED6 pad 1: Net-(LED1-VDD) -> +5V
- LED6 pad 4: Net-(LED1-VSS) -> GND
- LED60 pad 1: Net-(LED46-VDD) -> +5V
- LED60 pad 4: Net-(LED46-VSS) -> GND
- LED61 pad 1: Net-(LED61-VDD) -> +5V
- LED61 pad 4: Net-(LED61-VSS) -> GND
- LED62 pad 1: Net-(LED61-VDD) -> +5V
- LED62 pad 4: Net-(LED61-VSS) -> GND
- LED63 pad 1: Net-(LED61-VDD) -> +5V
- LED63 pad 4: Net-(LED61-VSS) -> GND
- LED64 pad 1: Net-(LED61-VDD) -> +5V
- LED64 pad 4: Net-(LED61-VSS) -> GND
- LED65 pad 1: Net-(LED61-VDD) -> +5V
- LED65 pad 4: Net-(LED61-VSS) -> GND
- LED66 pad 1: Net-(LED61-VDD) -> +5V
- LED66 pad 4: Net-(LED61-VSS) -> GND
- LED67 pad 1: Net-(LED61-VDD) -> +5V
- LED67 pad 4: Net-(LED61-VSS) -> GND
- LED68 pad 1: Net-(LED61-VDD) -> +5V
- LED68 pad 4: Net-(LED61-VSS) -> GND
- LED69 pad 1: Net-(LED61-VDD) -> +5V
- LED69 pad 4: Net-(LED61-VSS) -> GND
- LED7 pad 1: Net-(LED1-VDD) -> +5V
- LED7 pad 4: Net-(LED1-VSS) -> GND
- LED70 pad 1: Net-(LED61-VDD) -> +5V
- LED70 pad 4: Net-(LED61-VSS) -> GND
- LED71 pad 1: Net-(LED61-VDD) -> +5V
- LED71 pad 4: Net-(LED61-VSS) -> GND
- LED72 pad 1: Net-(LED61-VDD) -> +5V
- LED72 pad 4: Net-(LED61-VSS) -> GND
- LED73 pad 1: Net-(LED61-VDD) -> +5V
- LED73 pad 4: Net-(LED61-VSS) -> GND
- LED74 pad 1: Net-(LED61-VDD) -> +5V
- LED74 pad 4: Net-(LED61-VSS) -> GND
- LED75 pad 1: Net-(LED61-VDD) -> +5V
- LED75 pad 4: Net-(LED61-VSS) -> GND
- LED76 pad 1: Net-(LED76-VDD) -> +5V
- LED76 pad 4: Net-(LED76-VSS) -> GND
- LED77 pad 1: Net-(LED76-VDD) -> +5V
- LED77 pad 4: Net-(LED76-VSS) -> GND
- LED78 pad 1: Net-(LED76-VDD) -> +5V
- LED78 pad 4: Net-(LED76-VSS) -> GND
- LED79 pad 1: Net-(LED76-VDD) -> +5V
- LED79 pad 4: Net-(LED76-VSS) -> GND
- LED8 pad 1: Net-(LED1-VDD) -> +5V
- LED8 pad 4: Net-(LED1-VSS) -> GND
- LED80 pad 1: Net-(LED76-VDD) -> +5V
- LED80 pad 4: Net-(LED76-VSS) -> GND
- LED81 pad 1: Net-(LED76-VDD) -> +5V
- LED81 pad 4: Net-(LED76-VSS) -> GND
- LED82 pad 1: Net-(LED76-VDD) -> +5V
- LED82 pad 4: Net-(LED76-VSS) -> GND
- LED83 pad 1: Net-(LED76-VDD) -> +5V
- LED83 pad 4: Net-(LED76-VSS) -> GND
- LED84 pad 1: Net-(LED76-VDD) -> +5V
- LED84 pad 4: Net-(LED76-VSS) -> GND
- LED85 pad 1: Net-(LED76-VDD) -> +5V
- LED85 pad 4: Net-(LED76-VSS) -> GND
- LED86 pad 1: Net-(LED76-VDD) -> +5V
- LED86 pad 4: Net-(LED76-VSS) -> GND
- LED87 pad 1: Net-(LED76-VDD) -> +5V
- LED87 pad 4: Net-(LED76-VSS) -> GND
- LED9 pad 1: Net-(LED1-VDD) -> +5V
- LED9 pad 4: Net-(LED1-VSS) -> GND
Routing:
- net +5V: track 0.00 -> 2190.4 mm
- net GND: track 0.00 -> 2071.6 mm
- net Net-(LED16-DOUT): track 0.00 -> 381.7 mm
- net Net-(LED33-DOUT): track 0.00 -> 365.6 mm
- net Net-(LED50-DOUT): track 0.00 -> 364.7 mm
- net Net-(LED76-VSS): track 356.6 -> 0.00 mm
- net Net-(LED76-DOUT): track 0.00 -> 354.7 mm
- net Net-(LED1-VDD): track 328.9 -> 0.00 mm
- net Net-(LED76-VDD): track 327.8 -> 0.00 mm
- net Net-(LED63-DOUT): track 0.00 -> 285.2 mm
- net row2: track 336.4 -> 374.4 mm
- net row1: track 341.1 -> 379.2 mm
- net row0: track 340.4 -> 377.9 mm
- net Net-(D87-A): track 56.9 -> 85.5 mm
- net Net-(D82-A): track 56.9 -> 85.5 mm
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