File: keyboard_pcb/keyboard_pcb.kicad_pcb (KiCad board)
At the start: 2 copper layers, 360 x 140 mm, 373 parts, among them U1 NCP1117-3.3_SOT223, U2 RP2040, U3 W25Q128JVS

Commit message: started routing mcu
Parts:
- added D88: LED, LED_SMD:LED_0603_1608Metric_Pad1.05x0.95mm_HandSolder, B.Cu at (191.8, 216.5)
- added J1: USB_C_Receptacle_USB2.0_16P, Connector_USB:USB_C_Receptacle_GCT_USB4105-xx-A_16P_TopMnt_Horizontal, B.Cu at (57.7, 25.1)
- added J2: Conn_01x02, Connector_JST:JST_EH_B2B-EH-A_1x02_P2.50mm_Vertical, B.Cu at (179.5, 217.9)
- added R1: R, Resistor_SMD:R_0603_1608Metric_Pad0.98x0.95mm_HandSolder, B.Cu at (141.8, 152.4)
- added R2: 27, Resistor_SMD:R_0603_1608Metric_Pad0.98x0.95mm_HandSolder, B.Cu at (185.2, 201.2)
- added R3: 5.1k, Resistor_SMD:R_0603_1608Metric_Pad0.98x0.95mm_HandSolder, B.Cu at (185.2, 203.7)
- added R4: 27, Resistor_SMD:R_0603_1608Metric_Pad0.98x0.95mm_HandSolder, B.Cu at (185.2, 206.3)
- added R5: 5.1k, Resistor_SMD:R_0603_1608Metric_Pad0.98x0.95mm_HandSolder, B.Cu at (185.2, 208.8)
- added R6: 1k, Resistor_SMD:R_0603_1608Metric_Pad0.98x0.95mm_HandSolder, B.Cu at (185.2, 211.3)
- added R7: 1k, Resistor_SMD:R_0603_1608Metric_Pad0.98x0.95mm_HandSolder, B.Cu at (185.2, 213.8)
- added R8: 470, Resistor_SMD:R_0603_1608Metric_Pad0.98x0.95mm_HandSolder, B.Cu at (185.2, 216.3)
- added R9: 300, Resistor_SMD:R_0603_1608Metric_Pad0.98x0.95mm_HandSolder, B.Cu at (194.2, 210.4)
- added SW1: Reset, Button_Switch_SMD:SW_SPST_Omron_B3FS-100xP, B.Cu at (177.4, 211.4)
- added Y1: Crystal_GND24, Crystal:Crystal_SMD_Abracon_ABM8G-4Pin_3.2x2.5mm, B.Cu at (170.9, 217.5)
- U1, U2, U3: moved to B.Cu
- moved U2 202.1 mm to (129.5, 149.4), turned to 45 degrees
- moved U3 51.6 mm to (-49.0, -22.9), turned to 180 degrees
- moved U1 51.1 mm to (-48.8, -15.3), turned to 180 degrees
Connections:
- U2 pad 35: unconnected-(U2-GPIO23-Pad35) -> Net-(U2-GPIO23)
Routing:
- net row0: track 377.9 -> 596.2 mm
- net row1: track 379.2 -> 567.7 mm
- net row2: track 374.4 -> 544.7 mm
- net row3: track 285.6 -> 436.7 mm
- net row4: track 335.6 -> 475.1 mm
- net row5: track 358.1 -> 467.7 mm
- net col0: track 113.7 -> 207.1 mm, vias 0 -> 1
- net col1: track 87.0 -> 155.8 mm, vias 0 -> 1
- net col3: track 99.5 -> 149.7 mm, vias 0 -> 1
- net col5: track 99.5 -> 146.5 mm, vias 0 -> 1
- net col2: track 115.6 -> 159.6 mm, vias 0 -> 1
- net col4: track 99.5 -> 132.4 mm, vias 0 -> 1
- net col9: track 104.3 -> 107.4 mm, vias 0 -> 1
- net col8: track 103.5 -> 106.3 mm, vias 0 -> 1
- net col7: track 129.8 -> 132.1 mm, vias 0 -> 1
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