File: keyboard_pcb/matrix.kicad_sch (KiCad schematic)
At the start: 174 parts

Commit message: implemented LEDs and switch and diode layout
Parts:
- added S1: MX_stab, PCM_marbastlib-mx:STAB_MX_P_6.25u, symbol PCM_marbastlib-mx:MX_stab
- added S2: MX_stab, PCM_marbastlib-mx:STAB_MX_P_2.75u, symbol PCM_marbastlib-mx:MX_stab
- added S3, S5: MX_stab, PCM_marbastlib-mx:STAB_MX_P_2.25u, symbol PCM_marbastlib-mx:MX_stab
- added S6: MX_stab, PCM_marbastlib-mx:STAB_MX_P_2u, symbol PCM_marbastlib-mx:MX_stab
- renumbered D2 to D1, D11 to D10, D12 to D11, D13 to D12, D14 to D13, D15 to D14, D16 to D15, D17 to D16, D18 to D17, D19 to D18, D20 to D19, D3 to D2, D21 to D20, D22 to D21, D23 to D22, D24 to D23, D25 to D24, D26 to D25, D27 to D26, D28 to D27, D29 to D28, D30 to D29, D4 to D3, D31 to D30, D32 to D31, D33 to D32, D34 to D33, D35 to D34, D36 to D35, D37 to D36, D38 to D37, D39 to D38, D40 to D39, D5 to D4, D41 to D40, D42 to D41, D43 to D42, D44 to D43, D45 to D44, D46 to D45, D47 to D46, D48 to D47, D49 to D48, D50 to D49, D6 to D5, D51 to D50, D52 to D51, D53 to D52, D54 to D53, D55 to D54, D56 to D55, D57 to D56, D58 to D57, D59 to D58, D60 to D59, D7 to D6, D61 to D60, D62 to D61, D63 to D62, D64 to D63, D65 to D64, D66 to D65, D67 to D66, D68 to D67, D69 to D68, D70 to D69, D8 to D7, D71 to D70, D72 to D71, D73 to D72, D74 to D73, D75 to D74, D76 to D75, D77 to D76, D78 to D77, D79 to D78, D80 to D79, D9 to D8, D81 to D80, D82 to D81, D83 to D82, D84 to D83, D85 to D84, D86 to D85, D87 to D86, D88 to D87, D10 to D9
Connections:
- net col1: no longer D1.1 (K), D10.1 (K), D11.1 (K), D12.1 (K), D13.1 (K), D14.1 (K), D15.1 (K), D16.1 (K), D2.1 (K), D3.1 (K), D4.1 (K), D5.1 (K), D6.1 (K), D7.1 (K), D8.1 (K), D9.1 (K)
- net col16: no longer D51.1 (K), D52.1 (K), D53.1 (K), D54.1 (K), D55.1 (K), D56.1 (K), D57.1 (K), D58.1 (K), D59.1 (K), D60.1 (K), D61.1 (K), D62.1 (K), D63.1 (K), D64.1 (K), D65.1 (K), D66.1 (K), D67.1 (K), D68.1 (K), D69.1 (K), D70.1 (K), D71.1 (K), D72.1 (K), D73.1 (K), D74.1 (K), D75.1 (K), D76.1 (K)
- net col3: no longer D77.1 (K), D78.1 (K), D79.1 (K), D80.1 (K), D81.1 (K), D82.1 (K), D83.1 (K), D84.1 (K), D85.1 (K), D86.1 (K), D87.1 (K), MX21.1, MX22.1, MX23.1, MX25.1, MX26.1, MX38.1, MX39.1, MX4.1, MX40.1, MX42.1, MX43.1, MX5.1, MX54.1, MX55.1, MX56.1, MX58.1, MX59.1, MX6.1, MX67.1, MX68.1, MX69.1, MX71.1, MX72.1, MX8.1, MX9.1
- new net col4: MX21.1, MX38.1, MX4.1, MX54.1, MX67.1
- new net col5: MX22.1, MX39.1, MX5.1, MX55.1, MX68.1
- new net col6: MX23.1, MX40.1, MX56.1, MX6.1, MX69.1
- new net col8: MX25.1, MX42.1, MX58.1, MX71.1, MX8.1
- new net col9: MX26.1, MX43.1, MX59.1, MX72.1, MX9.1
- new net row0: D1.1 (K), D10.1 (K), D11.1 (K), D12.1 (K), D13.1 (K), D14.1 (K), D15.1 (K), D16.1 (K), D2.1 (K), D3.1 (K), D4.1 (K), D5.1 (K), D6.1 (K), D7.1 (K), D8.1 (K), D9.1 (K)
- new net row3: D51.1 (K), D52.1 (K), D53.1 (K), D54.1 (K), D55.1 (K), D56.1 (K), D57.1 (K), D58.1 (K), D59.1 (K), D60.1 (K), D61.1 (K), D62.1 (K), D63.1 (K)
- new net row4: D64.1 (K), D65.1 (K), D66.1 (K), D67.1 (K), D68.1 (K), D69.1 (K), D70.1 (K), D71.1 (K), D72.1 (K), D73.1 (K), D74.1 (K), D75.1 (K), D76.1 (K)
- new net row5: D77.1 (K), D78.1 (K), D79.1 (K), D80.1 (K), D81.1 (K), D82.1 (K), D83.1 (K), D84.1 (K), D85.1 (K), D86.1 (K), D87.1 (K)
Other:
- note added: "s6 for mx30"

Commit message: starting routing traces part 7
Connections:
- net col1: now also MX52.1
- net col2: no longer MX52.1
Other:
- moved on the sheet: D52, MX52
Changed lines of the file:
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@@
 	)
 	(junction
-		(at 86.36 111.76)
-		(diameter 0)
-		(color 0 0 0 0)
-	)
-	(junction
 		(at 229.87 77.47)
 		(diameter 0)
@@
 	)
 	(junction
-		(at 81.28 99.06)
-		(diameter 0)
-		(color 0 0 0 0)
-	)
-	(junction
 		(at 132.08 90.17)
 		(diameter 0)
@@
 	)
 	(junction
+		(at 69.85 99.06)
+		(diameter 0)
+		(color 0 0 0 0)
+	)
+	(junction
 		(at 109.22 90.17)
 		(diameter 0)
@@
 	)
 	(junction
+		(at 74.93 111.76)
+		(diameter 0)
+		(color 0 0 0 0)
+	)
+	(junction
 		(at 189.23 154.94)
 		(diameter 0)
@@
 	(wire
 		(pts
+			(xy 69.85 99.06) (xy 69.85 142.24)
+		)
+		(stroke
+			(width 0)
+			(type default)
+		)
+	)
+	(wire
+		(pts
 			(xy 62.23 154.94) (xy 74.93 154.94)
 		)
@@
 	(wire
 		(pts
-			(xy 62.23 111.76) (xy 86.36 111.76)
+			(xy 62.23 111.76) (xy 74.93 111.76)
 		)
 		(stroke
@@
 	(wire
 		(pts
+			(xy 74.93 111.76) (xy 97.79 111.76)
+		)
+		(stroke
+			(width 0)
+			(type default)
+		)
+	)
+	(wire
+		(pts
 			(xy 172.72 77.47) (xy 172.72 55.88)
 		)
@@
 	(wire
 		(pts
-			(xy 69.85 77.47) (xy 69.85 142.24)
+			(xy 69.85 77.47) (xy 69.85 99.06)
 		)
 		(stroke
@@
 	(wire
 		(pts
-			(xy 81.28 99.06) (xy 81.28 77.47)
+			(xy 81.28 77.47) (xy 81.28 120.65)
 		)
 		(stroke
@@
 	(wire
 		(pts
-			(xy 81.28 120.65) (xy 81.28 99.06)
-		)
-		(stroke
-			(width 0)
-			(type default)
-		)
-	)
-	(wire
-		(pts
 			(xy 184.15 77.47) (xy 184.15 99.06)
 		)
@@
 	(wire
 		(pts
-			(xy 86.36 111.76) (xy 97.79 111.76)
-		)
-		(stroke
-			(width 0)
-			(type default)
-		)
-	)
-	(wire
-		(pts
 			(xy 195.58 77.47) (xy 195.58 55.88)
 		)
@@
 	(symbol
 		(lib_id "PCM_marbastlib-mx:MX_SW_HS_CPG151101S11")
-		(at 83.82 101.6 0)
+		(at 72.39 101.6 0)
 		(unit 1)
 		(exclude_from_sim no)
@@
 		(fields_autoplaced yes)
 		(property "Reference" "MX52"
-			(at 83.82 93.98 0)
+			(at 72.39 93.98 0)
 			(effects
 				(font
@@
 		)
 		(property "Value" "MX_SW_HS"
-			(at 83.82 96.52 0)
+			(at 72.39 96.52 0)
 			(effects
 				(font
@@
 		)
 		(property "Footprint" "PCM_marbastlib-mx:SW_MX_HS_CPG151101S11_1u"
-			(at 83.82 101.6 0)
+			(at 72.39 101.6 0)
 			(effects
 				(font
@@
 		)
 		(property "Datasheet" "~"
-			(at 83.82 101.6 0)
+			(at 72.39 101.6 0)
 			(effects
 				(font
@@
 		)
 		(property "Description" "Push button switch, normally open, two pins, 45° tilted, Kailh CPG151101S11 for Cherry MX style switches"
-			(at 83.82 101.6 0)
+			(at 72.39 101.6 0)
 			(effects
 				(font
@@
 	(symbol
 		(lib_id "Device:D")
-		(at 86.36 107.95 90)
+		(at 74.93 107.95 90)
 		(unit 1)
 		(exclude_from_sim no)
@@
 		(fields_autoplaced yes)
 		(property "Reference" "D52"
-			(at 88.9 106.6799 90)
+			(at 77.47 106.6799 90)
 			(effects
 				(font
@@
 		)
 		(property "Value" "D"
-			(at 88.9 109.2199 90)
+			(at 77.47 109.2199 90)
 			(effects
 				(font
@@
 		)
 		(property "Footprint" "Diode_SMD:D_SOD-123"
-			(at 86.36 107.95 0)
+			(at 74.93 107.95 0)
 			(effects
 				(font
@@
 		)
 		(property "Datasheet" "~"
-			(at 86.36 107.95 0)
+			(at 74.93 107.95 0)
 			(effects
 				(font
@@
 		)
 		(property "Description" "Diode"
-			(at 86.36 107.95 0)
+			(at 74.93 107.95 0)
 			(effects
 				(font
@@
 		)
 		(property "Sim.Device" "D"
-			(at 86.36 107.95 0)
+			(at 74.93 107.95 0)
 			(effects
 				(font
@@
 		)
 		(property "Sim.Pins" "1=K 2=A"
-			(at 86.36 107.95 0)
+			(at 74.93 107.95 0)
 			(effects
 				(font

Commit message: added led capacitors and route all leds
Parts:
- renumbered S6 to S1, S3 to S2, S2 to S3, S5 to S4, S1 to S5
Changed lines of the file:
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@@
 		(dnp no)
 		(fields_autoplaced yes)
-		(property "Reference" "S5"
+		(property "Reference" "S4"
 			(at 80.01 123.0629 0)
 			(effects
@@
 			(project ""
 				(path "/5a0b976f-d314-4fca-8ab0-732ea8a514fc/a8e39055-a26b-42b9-b581-42b61b3ed0e5"
-					(reference "S5")
+					(reference "S4")
 					(unit 1)
 				)
@@
 		(dnp no)
 		(fields_autoplaced yes)
-		(property "Reference" "S6"
+		(property "Reference" "S1"
 			(at 270.51 49.4029 0)
 			(effects
@@
 			(project ""
 				(path "/5a0b976f-d314-4fca-8ab0-732ea8a514fc/a8e39055-a26b-42b9-b581-42b61b3ed0e5"
-					(reference "S6")
+					(reference "S1")
 					(unit 1)
 				)
@@
 		(dnp no)
 		(fields_autoplaced yes)
-		(property "Reference" "S2"
+		(property "Reference" "S3"
 			(at 227.33 120.5229 0)
 			(effects
@@
 			(project ""
 				(path "/5a0b976f-d314-4fca-8ab0-732ea8a514fc/a8e39055-a26b-42b9-b581-42b61b3ed0e5"
-					(reference "S2")
+					(reference "S3")
 					(unit 1)
 				)
@@
 		(dnp no)
 		(fields_autoplaced yes)
-		(property "Reference" "S1"
+		(property "Reference" "S5"
 			(at 162.56 143.3829 0)
 			(effects
@@
 			(project ""
 				(path "/5a0b976f-d314-4fca-8ab0-732ea8a514fc/a8e39055-a26b-42b9-b581-42b61b3ed0e5"
-					(reference "S1")
+					(reference "S5")
 					(unit 1)
 				)
@@
 		(dnp no)
 		(fields_autoplaced yes)
-		(property "Reference" "S3"
+		(property "Reference" "S2"
 			(at 229.87 100.2029 0)
 			(effects
@@
 			(project ""
 				(path "/5a0b976f-d314-4fca-8ab0-732ea8a514fc/a8e39055-a26b-42b9-b581-42b61b3ed0e5"
-					(reference "S3")
+					(reference "S2")
 					(unit 1)
 				)
